File: pcb/hackpad2.kicad_sch (KiCad schematic)
At the start: 26 parts, among them SW10 SW_Push, SW11 SW_Push, SW12 SW_Push, SW13 SW_Push, SW2 SW_Push, SW3 SW_Push, SW4 SW_Push, SW5 SW_Push, SW6 SW_Push, SW7 SW_Push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

Commit message: journal 1
Connections:
- net GND: now also U2.1 (GND); no longer U2.2 (VCC)
- net VCC: now also U2.2 (VCC); no longer U2.1 (GND)
- net row2: now reaches D5.1 (K), D6.1 (K), D7.1 (K), D8.1 (K)
- net row2: now also U1.9 (PA7_A8_D8_SCK)
- net row0: now reaches D4.1 (K)
- net row0: now also D12.1 (K), D13.1 (K), D2.1 (K), U1.11 (PA6_A10_D10_MOSI)
- net row1: now reaches D9.1 (K)
- net row1: now also D10.1 (K), D11.1 (K), D3.1 (K), U1.10 (PA5_A9_D9_MISO)

Commit message: schematic done?
Parts:
- removed D12, D8, D9: D_Small, symbol Device:D_Small
- removed SW12, SW8, SW9: SW_Push, symbol Switch:SW_Push
- added D1, D12, D14, D15, D16, D17, D18, D8, D9: SK6812MINI-E, LED_SMD:LED_SK6812MINI-E_3.2x2.8mm_P1.5mm_ReverseMount, symbol LED:SK6812MINI-E
- added SW1: RotaryEncoder_Switch, symbol Device:RotaryEncoder_Switch
Connections:
- net GND: now also D1.1 (VSS), D12.1 (VSS), D14.1 (VSS), D15.1 (VSS), D16.1 (VSS), D17.1 (VSS), D18.1 (VSS), D8.1 (VSS), D9.1 (VSS), SW1.C, SW1.S2
- net VCC: now also D1.3 (VDD), D12.3 (VDD), D14.3 (VDD), D15.3 (VDD), D16.3 (VDD), D17.3 (VDD), D18.3 (VDD), D8.3 (VDD), D9.3 (VDD)
- net RE_SW: now reaches U1.7 (PB08_A6_D6_TX)
- net RE_SW: now also SW1.S1
- net RE2: now reaches U1.8 (PB09_A7_D7_RX)
- net RE2: now also SW1.B
- net col4 renamed leds
- net leds: now also D1.2 (DIN)
- new net: D14.4 (DOUT), D15.2 (DIN)
- new net: D15.4 (DOUT), D16.2 (DIN)
- new net: D16.4 (DOUT), D17.2 (DIN)
- new net: D17.4 (DOUT), D18.2 (DIN)
- new net: D12.4 (DOUT), D14.2 (DIN)
- new net: D1.4 (DOUT), D8.2 (DIN)
- new net: D8.4 (DOUT), D9.2 (DIN)
- new net: D12.2 (DIN), D9.4 (DOUT)
- new net RE1: SW1.A
Other:
- moved on the sheet: D10, D11, D13, D2, D3, D4, D5, D6, D7, SW10, SW11, SW13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

Commit message: routing
Parts:
- D10, D11, D13, D2, D3, D4, D5, D6, D7: footprint (none) -> Diode_THT:D_DO-35_SOD27_P7.62mm_Horizontal
- SW1: footprint (none) -> Rotary_Encoder:RotaryEncoder_Alps_EC11E-Switch_Vertical_H20mm
- SW10, SW11, SW13, SW2, SW3, SW4, SW5, SW6, SW7: footprint (none) -> Button_Switch_Keyboard:SW_Cherry_MX_1.00u_PCB
- U1: footprint (none) -> footprints:XIAO-Generic-Hybrid-14P-2.54-21X17.8MM
Changed lines of the file:
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@@
 			)
 		)
-		(property "Footprint" ""
+		(property "Footprint" "Rotary_Encoder:RotaryEncoder_Alps_EC11E-Switch_Vertical_H20mm"
 			(at 53.34 32.766 0)
 			(hide yes)
@@
 			)
 		)
-		(property "Footprint" ""
+		(property "Footprint" "Diode_THT:D_DO-35_SOD27_P7.62mm_Horizontal"
 			(at 74.93 181.61 90)
 			(hide yes)
@@
 			)
 		)
-		(property "Footprint" ""
+		(property "Footprint" "Button_Switch_Keyboard:SW_Cherry_MX_1.00u_PCB"
 			(at 54.61 135.89 0)
 			(hide yes)
@@
 			)
 		)
-		(property "Footprint" ""
+		(property "Footprint" "Button_Switch_Keyboard:SW_Cherry_MX_1.00u_PCB"
 			(at 86.36 156.21 0)
 			(hide yes)
@@
 			)
 		)
-		(property "Footprint" ""
+		(property "Footprint" "Diode_THT:D_DO-35_SOD27_P7.62mm_Horizontal"
 			(at 74.93 140.97 90)
 			(hide yes)
@@
 			)
 		)
-		(property "Footprint" ""
+		(property "Footprint" "Button_Switch_Keyboard:SW_Cherry_MX_1.00u_PCB"
 			(at 86.36 176.53 0)
 			(hide yes)
@@
 			)
 		)
-		(property "Footprint" ""
+		(property "Footprint" "Diode_THT:D_DO-35_SOD27_P7.62mm_Horizontal"
 			(at 43.18 140.97 90)
 			(hide yes)
@@
 			)
 		)
-		(property "Footprint" ""
+		(property "Footprint" "Diode_THT:D_DO-35_SOD27_P7.62mm_Horizontal"
 			(at 38.1 181.61 90)
 			(hide yes)
@@
 			)
 		)
-		(property "Footprint" ""
+		(property "Footprint" "Button_Switch_Keyboard:SW_Cherry_MX_1.00u_PCB"
 			(at 49.53 176.53 0)
 			(hide yes)
@@
 			)
 		)
-		(property "Footprint" ""
+		(property "Footprint" "Button_Switch_Keyboard:SW_Cherry_MX_1.00u_PCB"
 			(at 120.65 176.53 0)
 			(hide yes)
@@
 			)
 		)
-		(property "Footprint" ""
+		(property "Footprint" "Diode_THT:D_DO-35_SOD27_P7.62mm_Horizontal"
 			(at 43.18 161.7352 90)
 			(hide yes)
@@
 			)
 		)
-		(property "Footprint" ""
+		(property "Footprint" "footprints:XIAO-Generic-Hybrid-14P-2.54-21X17.8MM"
 			(at 44.45 67.31 0)
 			(hide yes)
@@
 			)
 		)
-		(property "Footprint" ""
+		(property "Footprint" "Diode_THT:D_DO-35_SOD27_P7.62mm_Horizontal"
 			(at 74.93 161.29 90)
 			(hide yes)
@@
 			)
 		)
-		(property "Footprint" ""
+		(property "Footprint" "Button_Switch_Keyboard:SW_Cherry_MX_1.00u_PCB"
 			(at 86.36 135.89 0)
 			(hide yes)
@@
 			)
 		)
-		(property "Footprint" ""
+		(property "Footprint" "Diode_THT:D_DO-35_SOD27_P7.62mm_Horizontal"
 			(at 109.22 143.51 90)
 			(hide yes)
@@
 			)
 		)
-		(property "Footprint" ""
+		(property "Footprint" "Button_Switch_Keyboard:SW_Cherry_MX_1.00u_PCB"
 			(at 54.61 156.6552 0)
 			(hide yes)
@@
 			)
 		)
-		(property "Footprint" ""
+		(property "Footprint" "Diode_THT:D_DO-35_SOD27_P7.62mm_Horizontal"
 			(at 109.22 181.61 90)
 			(hide yes)
@@
 			)
 		)
-		(property "Footprint" ""
+		(property "Footprint" "Button_Switch_Keyboard:SW_Cherry_MX_1.00u_PCB"
 			(at 120.65 138.43 0)
 			(hide yes)
@@
 			)
 		)
-		(property "Footprint" ""
+		(property "Footprint" "Button_Switch_Keyboard:SW_Cherry_MX_1.00u_PCB"
 			(at 120.65 154.94 0)
 			(hide yes)
@@
 			)
 		)
-		(property "Footprint" ""
+		(property "Footprint" "Diode_THT:D_DO-35_SOD27_P7.62mm_Horizontal"
 			(at 109.22 160.02 90)
 			(hide yes)
