File: pcb/hackpad2.kicad_pcb (KiCad board)
At the start: 2 copper layers, 3.6 x 3.2 mm, 30 parts, among them SW1 RotaryEncoder_Switch, SW10 SW_Push, SW11 SW_Push, SW13 SW_Push, SW2 SW_Push, SW3 SW_Push, SW4 SW_Push, SW5 SW_Push, SW6 SW_Push, SW7 SW_Push, U1 MOUDLE-SEEEDUINO-XIAO, U2 ER_OLEDM0.91_1x-I2C

Commit message: ROUTING DONE
Parts:
- moved D13 44.0 mm to (83.7, 48.5)
- moved D5 41.5 mm to (83.9, 93.0)
- moved D4 32.0 mm to (83.8, 52.5)
- moved D10 17.0 mm to (83.9, 72.5)
- moved D6 12.0 mm to (83.9, 88.5)
- moved D2 9.00 mm to (83.9, 56.5)
- moved D7 4.50 mm to (84.0, 84.0)
- moved D3 3.00 mm to (83.9, 76.0)
- moved D11 0.50 mm to (83.9, 79.5)
- moved SW6 0.16 mm to (124.5, 85.9)
- moved SW7 0.16 mm to (143.5, 86.0)
- moved SW2 0.14 mm to (105.5, 47.9)
- moved SW11 0.09 mm to (105.5, 66.9)
- moved SW4 0.08 mm to (124.5, 47.9)
Connections:
- SW1 pad S1: RE_SW -> unconnected-(SW1-PadS1)
- SW1 pad S2: GND -> unconnected-(SW1-PadS2)
- U1 pad 1: col0 -> col2
- U1 pad 10: row1 -> row2
- U1 pad 3: col2 -> col0
- U1 pad 7: RE_SW -> RE1
- U1 pad 9: row2 -> row1
Routing:
- net GND: track 0.00 -> 354.9 mm
- net VCC: track 0.00 -> 312.9 mm
- net col2: track 0.00 -> 141.6 mm
- net col1: track 0.00 -> 110.9 mm
- net col0: track 0.00 -> 87.9 mm
- net row0: track 0.00 -> 74.4 mm
- net Net-(D12-DIN): track 0.00 -> 61.2 mm
- net Net-(D15-DOUT): track 0.00 -> 60.5 mm
- net Net-(D10-A): track 0.00 -> 55.8 mm
- net Net-(D13-A): track 0.00 -> 54.0 mm
- net Net-(D7-A): track 0.00 -> 52.7 mm
- net leds: track 0.00 -> 48.6 mm
- net row1: track 0.00 -> 39.0 mm
- net Net-(D3-A): track 0.00 -> 38.7 mm
- net Net-(D4-A): track 0.00 -> 36.1 mm
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
Commit message: silkscreen
Other:
- board size 3.6 x 3.2 mm -> 107.5 x 61 mm
